File: hardware/MitsubishiSC.kicad_pcb (KiCad board)
At the start: 6 copper layers, 30 x 50 mm, 68 parts, among them J1 CN105, J2 USB_C_Receptacle_USB2.0_16P, Q1 BSS138, Q2 BSS138, SW3 SPST, SW4 SPST, U1 TPS562203, U3 ESP32-C3-WROOM-02, U4 USBLC6-2SC6, U5 TLV75733PDBV

Commit message: fix(hw): swap C6/C17 cap placement
This commit fixes an issue with the SMPS output cap placement where the
100nF capacitor should have been placed closest to the pins but is not
the case.
Parts:
- moved C17 3.00 mm to (155.2, 104.0)
- moved C6 3.00 mm to (152.2, 104.0)
Changed lines of the file:
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@@
 	(footprint "Capacitor_SMD:C_0603_1608Metric"
 		(layer "F.Cu")
-		(at 152.15 104 90)
+		(at 155.15 104 90)
 		(descr "Capacitor SMD 0603 (1608 Metric), square (rectangular) end terminal, IPC_7351 nominal, (Body size source: IPC-SM-782 page 76, https://www.pcb-3d.com/wordpress/wp-content/uploads/ipc-sm-782a_amendment_1_and_2.pdf), generated with kicad-footprint-generator")
 		(tags "capacitor")
@@
 	(footprint "Capacitor_SMD:C_0603_1608Metric"
 		(layer "F.Cu")
-		(at 155.15 104 90)
+		(at 152.15 104 90)
 		(descr "Capacitor SMD 0603 (1608 Metric), square (rectangular) end terminal, IPC_7351 nominal, (Body size source: IPC-SM-782 page 76, https://www.pcb-3d.com/wordpress/wp-content/uploads/ipc-sm-782a_amendment_1_and_2.pdf), generated with kicad-footprint-generator")
 		(tags "capacitor")

Commit message: feat(hw): reduce LED brightness
This commit reduces the brightness of the indicator LED by increasing
the resistor value of R8 from 1kR to 10kR. Although the resistor value
is on the higher side, this is generally fine because the use of LED is
not user-facing.
Parts:
- R8: value 1kR -> 10kR
Changed lines of the file:
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@@
 			)
 		)
-		(property "Value" "1kR"
+		(property "Value" "10kR"
 			(at 0 1.43 0)
 			(layer "F.Fab")
@@
 			)
 		)
-		(property "Datasheet" "https://www.lcsc.com/datasheet/lcsc_datasheet_2304140030_YAGEO-RC0603FR-071KL_C22548.pdf"
+		(property "Datasheet" "https://www.lcsc.com/datasheet/lcsc_datasheet_2304140030_YAGEO-RC0603FR-0710KL_C98220.pdf"
 			(at 0 0 180)
 			(unlocked yes)
@@
 			)
 		)
-		(property "Distributor Part Number" "C22548"
+		(property "Distributor Part Number" "C98220"
 			(at 0 0 180)
 			(unlocked yes)
@@
 			)
 		)
-		(property "Manufacturer Part Number" "RC0603FR-071KL"
+		(property "Manufacturer Part Number" "RC0603FR-0710KL"
 			(at 0 0 180)
 			(unlocked yes)

Commit message: fix(hw): incorrect PPTC footprint
This commit fixes the incorrect PPTC footprint size.

The existing schematic specifies the Bourns MF-MSMF030-2 part which
should be using the `Fuse_1812_4532Metric` footprint but was instead
assigned the `Fuse_1206_3216Metric` footprint. As a result, the
component CANNOT be placed on the circuit board.

To rectify this, we changed the component to use the Littelfuse
1206L035/16 part instead, which is almost similar to the specifications
of the original part.

Importantly, a deliberate decision was made to swap component instead of
correcting the footprint in order to avoid the significant change to the
board layout required to accommodate the correct but larger 1812
footprint.
Parts:
- F1, F2: value 300mA -> 350mA
Changed lines of the file:
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@@
 			)
 		)
-		(property "Value" "300mA"
+		(property "Value" "350mA"
 			(at 0 1.82 90)
 			(layer "F.Fab")
@@
 			)
 		)
-		(property "Datasheet" "https://www.lcsc.com/datasheet/lcsc_datasheet_1808271848_BOURNS-MF-MSMF030-2_C12604.pdf"
+		(property "Datasheet" "https://www.lcsc.com/datasheet/C126817.pdf"
 			(at 0 0 90)
 			(unlocked yes)
@@
 			)
 		)
-		(property "Distributor Part Number" "C12604"
+		(property "Distributor Part Number" "C126817"
 			(at 0 0 90)
 			(unlocked yes)
@@
 			)
 		)
-		(property "Manufacturer" "Bourns Inc."
+		(property "Manufacturer" "Littelfuse"
 			(at 0 0 90)
 			(unlocked yes)
@@
 			)
 		)
-		(property "Manufacturer Part Number" "MF-MSMF030-2"
+		(property "Manufacturer Part Number" "1206L035/16"
 			(at 0 0 90)
 			(unlocked yes)
@@
 			)
 		)
-		(property "Value" "300mA"
+		(property "Value" "350mA"
 			(at 0 1.82 90)
 			(layer "F.Fab")
@@
 			)
 		)
-		(property "Datasheet" "https://www.lcsc.com/datasheet/lcsc_datasheet_1808271848_BOURNS-MF-MSMF030-2_C12604.pdf"
+		(property "Datasheet" "https://www.lcsc.com/datasheet/C126817.pdf"
 			(at 0 0 90)
 			(unlocked yes)
@@
 			)
 		)
-		(property "Distributor Part Number" "C12604"
+		(property "Distributor Part Number" "C126817"
 			(at 0 0 90)
 			(unlocked yes)
@@
 			)
 		)
-		(property "Manufacturer" "Bourns Inc."
+		(property "Manufacturer" "Littelfuse"
 			(at 0 0 90)
 			(unlocked yes)
@@
 			)
 		)
-		(property "Manufacturer Part Number" "MF-MSMF030-2"
+		(property "Manufacturer Part Number" "1206L035/16"
 			(at 0 0 90)
 			(unlocked yes)
