File: hardware/MitsubishiSC.kicad_pcb (KiCad board)
At the start: 6 copper layers, 50 x 43 mm, 66 parts, among them J1 CN105, J2 TC2050, Q1 BSS138, Q2 BSS138, SW1 SPST, SW2 SPST, U1 ESP32-C6-WROOM-1, U2 TPS54202DDC, U3 TLV75733PDBV, U4 USBLC6-2SC6

Commit message: feat: upgrade project to KiCad 10 (#60)
Migrate the schematic, PCB and project files to the KiCad 10 format and
bump hardware/lib from ccd4174 to 341530d, which reorganises the custom
libraries into ZY_* KLC categories exposed through nested library
tables.

- Point sym-lib-table/fp-lib-table at the nested ZY tables via
  ${KIPRJMOD}/lib instead of the old _Custom entries
- Relink J1 to ZY_Connector:Mitsubishi_CN105_Device_MountingPin and
  JST_PA_SM05B-PASS_1x05-1MP_P2.00mm_Horizontal, wiring the new MP pin
  to GND to match the footprint's mounting pads
- Relink U1 to ZY_RF_Module:ESP32-C6-WROOM-1
- Restore Datasheet and Distributor/Manufacturer fields on J1 and U1
  that were dropped when changing symbols
- Exclude the F1/F2 footprint_filter errors newly reported by KiCad 10,
  as the stock Polyfuse filter doesn't match Fuse_1206
- Bump CI to kicad/kicad:10.0.7
Parts:
- J1: footprint _Custom:JST_PA_SM05B-PASS_1x05_P2.00mm_Horizontal -> ZY_Connector:JST_PA_SM05B-PASS_1x05-1MP_P2.00mm_Horizontal
- U1: footprint _Custom:ESP32-C6-WROOM-1 -> ZY_RF_Module:ESP32-C6-WROOM-1
